Commit message: Add: New URDF file with an attached lidar. Changes in the launch file to include bridge of both /scan and /odom. Fix: Errors that prevented spawning

File: install/claus_description/share/claus_description/urdf/accessories.urdf.xacro (robot description, xacro)
@@ -9,4 +9,40 @@
     ridgeback_base/launch/base.launch
   -->
+<xacro:macro name="simple_lidar" params="prefix parent_link location topic">
+  <link name="${prefix}_laser">
+    <visual>
+      <geometry>
+        <cylinder radius="0.05" length="0.05"/>
+      </geometry>
+      <material name="black"/>
+    </visual>
+  </link>
+  <joint name="${prefix}_laser_joint" type="fixed">
+    <parent link="${parent_link}"/>
+    <child link="${prefix}_laser"/>
+    <origin xyz="${location * 0.3999} 0 0.2337"
+            rpy="0 0 ${PI/2 - (location * PI/2)}"/>
+  </joint>
+  <gazebo reference="${prefix}_laser">
+    <sensor name="${prefix}_lidar" type="gpu_lidar">
+      <always_on>true</always_on>
+      <update_rate>10</update_rate>
+      <topic>${topic}</topic>
+      <ray>
+        <scan>
+          <horizontal>
+            <samples>720</samples>
+            <min_angle>-3.14</min_angle>
+            <max_angle>3.14</max_angle>
+          </horizontal>
+        </scan>
+        <range>
+          <min>0.1</min>
+          <max>20.0</max>
+        </range>
+      </ray>
+    </sensor>
+  </gazebo>
+</xacro:macro>
   <xacro:include filename="$(find claus_description)/urdf/accessories/sick_lms1xx_mount.urdf.xacro" />
   <xacro:include filename="$(find claus_description)/urdf/accessories/sick_s300_mount.urdf.xacro" />

File: install/claus_description/share/claus_description/urdf/ridgeback.urdf.xacro (robot description, xacro)
@@ -28,5 +28,5 @@
         <origin xyz="0 0 0" rpy="${PI/2} 0 0"/>
         <geometry>
-          <mesh filename="package://claus_description/meshes/wheel.stl"/>
+          <mesh filename="file://$(find claus_description)/meshes/wheel.stl"/>
         </geometry>
         <material name="black" />
@@ -68,5 +68,5 @@
         <origin xyz="0 0 0" rpy="${PI/2} 0 ${PI/2}" />
         <geometry>
-          <mesh filename="package://claus_description/meshes/rocker.stl"/>
+          <mesh filename="file://$(find claus_description)/meshes/rocker.stl"/>
         </geometry>
         <material name="black" />
@@ -111,5 +111,5 @@
       <origin xyz="0 0 0" rpy="0 0 0" />
       <geometry>
-        <mesh filename="package://claus_description/meshes/body.stl"/>
+        <mesh filename="file://$(find claus_description)/meshes/body.stl"/>
       </geometry>
       <material name="black" />
@@ -118,5 +118,5 @@
       <origin xyz="0 0 0"/>
       <geometry>
-        <mesh filename="package://claus_description/meshes/body-collision.stl"/>
+        <mesh filename="file://$(find claus_description)/meshes/body-collision.stl"/>
       </geometry>
     </collision>
@@ -164,5 +164,5 @@
       <origin xyz="0 0 0" rpy="0 0 ${PI}" />
       <geometry>
-        <mesh filename="package://claus_description/meshes/side-cover.stl"/>
+        <mesh filename="file://$(find claus_description)/meshes/side-cover.stl"/>
       </geometry>
       <material name="yellow" />
@@ -173,5 +173,5 @@
       <origin xyz="0 0 0" rpy="0 0 0" />
       <geometry>
-        <mesh filename="package://claus_description/meshes/side-cover.stl"/>
+        <mesh filename="file://$(find claus_description)/meshes/side-cover.stl"/>
       </geometry>
       <material name="yellow" />
@@ -187,5 +187,5 @@
       <origin xyz="0 0 0" rpy="0 0 0" />
       <geometry>
-        <mesh filename="package://claus_description/meshes/end-cover.stl" />
+        <mesh filename="file://$(find claus_description)/meshes/end-cover.stl" />
       </geometry>
       <material name="black" />
@@ -201,5 +201,5 @@
       <origin xyz="0 0 0" rpy="0 0 ${PI}" />
       <geometry>
-        <mesh filename="package://claus_description/meshes/end-cover.stl" />
+        <mesh filename="file://$(find claus_description)/meshes/end-cover.stl" />
       </geometry>
       <material name="black" />
@@ -220,5 +220,5 @@
       <origin xyz="0 0 0" rpy="0 0 0" />
       <geometry>
-        <mesh filename="package://claus_description/meshes/lights.stl" />
+        <mesh filename="file://$(find claus_description)/meshes/lights.stl" />
       </geometry>
       <material name="white" />
@@ -229,5 +229,5 @@
       <origin xyz="0 0 0" rpy="0 0 ${PI}" />
       <geometry>
-        <mesh filename="package://claus_description/meshes/lights.stl" />
+        <mesh filename="file://$(find claus_description)/meshes/lights.stl" />
       </geometry>
       <material name="black" />
@@ -243,5 +243,5 @@
       <origin xyz="0 0 0" rpy="0 0 0" />
       <geometry>
-        <mesh filename="package://claus_description/meshes/top.stl" />
+        <mesh filename="file://$(find claus_description)/meshes/top.stl" />
       </geometry>
       <material name="black" />
@@ -250,5 +250,5 @@
       <origin xyz="0 0 0" rpy="0 0 0" />
       <geometry>
-        <mesh filename="package://claus_description/meshes/top.stl"/>
+        <mesh filename="file://$(find claus_description)/meshes/top.stl"/>
       </geometry>
     </collision>
@@ -263,5 +263,5 @@
       <origin xyz="0 0 0" rpy="0 ${PI/2} 0" />
       <geometry>
-        <mesh filename="package://claus_description/meshes/axle.stl" />
+        <mesh filename="file://$(find claus_description)/meshes/axle.stl" />
       </geometry>
       <material name="black" />
@@ -294,3 +294,15 @@
   <!-- Optional custom includes. -->
   <xacro:include filename="$(optenv RIDGEBACK_URDF_EXTRAS empty.urdf)" />
+  <!-- Front lidar -->
+  <xacro:simple_lidar
+    prefix="front"
+    parent_link="chassis_link"
+    location="1"
+    topic="scan"/>
+  <!-- Rear lidar -->
+  <xacro:simple_lidar
+    prefix="rear"
+    parent_link="chassis_link"
+    location="-1"
+    topic="rear/scan"/>
 </robot>
