Commit message: shoot me..... trying to make the r100 from clearpath to work, odometry works for that one, it already have a tf tree and build in sensors to use. Trying to make the lidar to work, however slam just dont want to publish map or scan_visualization

File: src/clearpath_common/clearpath_sensors_description/urdf/velodyne_lidar.urdf.xacro (robot description, xacro)
@@ -64,5 +64,5 @@
         <visualize>true</visualize>
         <always_on>true</always_on>
-        <gz_frame_id>${name}_laser</gz_frame_id>
+        <gz_frame_id>r100/${name}_laser</gz_frame_id>
         <topic>$(arg namespace)/sensors/${name}/scan</topic>
         <lidar>

File: src/lab_manipulator/urdf/r100_wrapper.xacro (robot description, xacro)
@@ -3,4 +3,7 @@
   <xacro:arg name="use_platform_controllers" default="false"/>
   <xacro:include filename="$(find clearpath_platform_description)/urdf/r100/r100.urdf.xacro"/>
+  <xacro:include filename="$(find claus_description)/urdf/accessories.urdf.xacro"/>
+  <xacro:property name="PI" value="3.1415926535897931"/> # Define PI for use in lidar for some reason
+  <xacro:include filename="$(find clearpath_sensors_description)/urdf/velodyne_lidar.urdf.xacro"/>
   <xacro:r100/>
    <gazebo>
@@ -15,3 +18,8 @@
     </plugin>
     </gazebo>
+  <xacro:velodyne_lidar
+    name="front_lidar"
+    parent_link="chassis_link">
+    <origin xyz="0.3999 0 0.2337" rpy="0 0 0"/>
+  </xacro:velodyne_lidar>
 </robot>
