Commit message: good luck

File: src/claus_sim/claus_description/urdf/accessories.urdf.xacro (robot description, xacro)
@@ -30,5 +30,5 @@
       <visualize>true</visualize>
       <topic>${topic}</topic>
-      <gz_frame_id>${prefix}_laser</gz_frame_id>
+      <gz_frame_id>r100/${prefix}_laser</gz_frame_id>
       <lidar>
         <scan>

File: src/lab_manipulator/urdf/r100_wrapper.xacro (robot description, xacro)
@@ -7,4 +7,9 @@
   <xacro:include filename="$(find clearpath_sensors_description)/urdf/velodyne_lidar.urdf.xacro"/>
   <xacro:r100/>
+    <xacro:simple_lidar
+      prefix="front"
+      parent_link="chassis_link"
+      location="1"
+      topic="/sensors/front_lidar/scan"/>
    <gazebo>
      <plugin filename="gz-sim-diff-drive-system" name="gz::sim::systems::DiffDrive">
@@ -18,8 +23,9 @@
     </plugin>
     </gazebo>
-  <xacro:velodyne_lidar
-    name="front_lidar"
-    parent_link="chassis_link">
-    <origin xyz="0.3999 0 0.2337" rpy="0 0 0"/>
-  </xacro:velodyne_lidar>
+    <gazebo>
+      <plugin filename="gz-sim-joint-state-publisher-system"
+              name="gz::sim::systems::JointStatePublisher">
+               <update_rate>50</update_rate>
+      </plugin>
+    </gazebo>
 </robot>
