Commit message: Clearpath ridgeback in empty world

File: src/clearpath_common/clearpath_platform_description/urdf/r100/r100.urdf.xacro (robot description, xacro)
@@ -5,4 +5,17 @@
   <xacro:arg name="gazebo_controllers" default="$(find clearpath_control)/config/r100/control/omni_4wd.yaml"/>
   <xacro:arg name="use_platform_controllers" default="true"/>
+  <!-- Self defined colors-->
+  <material name="clearpath_dark_grey">
+  <color rgba="0.25 0.25 0.25 1"/>
+  </material>
+  <material name="clearpath_black">
+    <color rgba="0.05 0.05 0.05 1"/>
+  </material>
+  <material name="clearpath_light_grey">
+    <color rgba="0.7 0.7 0.7 1"/>
+  </material>
+  <material name="clearpath_yellow">
+    <color rgba="1.0 0.8 0.0 1"/>
+  </material>
   <!-- R100 Platform Macro -->
   <xacro:macro name="r100" params="control:='omni_4wd' front_wheels:='mecanum' rear_wheels:='mecanum'">

Commit message: fix: update launch files and URDF configurations for improved simulation setup

File: src/clearpath_common/clearpath_platform_description/urdf/r100/r100.urdf.xacro (robot description, xacro)
@@ -17,4 +17,10 @@
   <material name="clearpath_yellow">
     <color rgba="1.0 0.8 0.0 1"/>
+  </material>
+  <material name="clearpath_white">
+    <color rgba="1.0 1.0 1.0 1"/>
+  </material>
+  <material name="clearpath_red">
+    <color rgba="1.0 0.0 0.0 1"/>
   </material>
   <!-- R100 Platform Macro -->

File: src/lab_manipulator/urdf/accessories.urdf.xacro (robot description, xacro)
@@ -7,5 +7,5 @@
           <cylinder radius="0.05" length="0.05"/>
         </geometry>
-        <material name="black"/>
+        <material name="clearpath_black"/>
       </visual>
     </link>

Commit message: Add: The SDL now has the top table. Still missing camera and manipulator

File: src/clearpath_common/clearpath_platform_description/urdf/r100/r100.urdf.xacro (robot description, xacro)
@@ -7,5 +7,5 @@
   <!-- Self defined colors-->
   <material name="clearpath_dark_grey">
-  <color rgba="0.25 0.25 0.25 1"/>
+    <color rgba="0.25 0.25 0.25 1"/>
   </material>
   <material name="clearpath_black">

File: src/lab_manipulator/urdf/r100_wrapper.xacro (robot description, xacro)
@@ -5,4 +5,27 @@
   <xacro:include filename="$(find clearpath_platform_description)/urdf/r100/r100.urdf.xacro"/>
   <xacro:include filename="$(find lab_manipulator)/urdf/accessories.urdf.xacro"/>
+  <material name="black">
+    <color rgba="0 0 0 1"/>
+  </material>
+  <link name="mounting_structure_link">
+    <visual>
+      <origin xyz="0 0 0" rpy="0 0 0"/>
+      <material name="black"/>
+      <geometry>
+        <mesh filename="package://lab_manipulator/meshes/mounting_structure.STL"/>
+      </geometry>
+    </visual>
+    <collision>
+      <origin xyz="0 0 0" rpy="0 0 0"/>
+      <geometry>
+        <mesh filename="package://lab_manipulator/meshes/mounting_structure.STL"/>
+      </geometry>
+    </collision>
+  </link>
+  <joint name="mounting_structure_joint" type="fixed">
+    <parent link="default_mount"/>
+    <child link="mounting_structure_link"/>
+    <origin xyz="0.0 0.0 -0.006" rpy="0 0 0"/>
+  </joint>
   <xacro:r100/>
     <xacro:simple_lidar
