Commit message: FIX: moved everything related to the physical robot (claus) into claus pkg from lab_manipulator. BUUUUUT i accidently removed the top part....

File: src/claus/urdf/r100_wrapper.xacro (robot description, xacro)
@@ -4,5 +4,5 @@
   <xacro:property name="PI" value="3.1415926535897931"/>
   <xacro:include filename="$(find clearpath_platform_description)/urdf/r100/r100.urdf.xacro"/>
-  <xacro:include filename="$(find lab_manipulator)/urdf/accessories.urdf.xacro"/>
+  <xacro:include filename="$(find claus)/urdf/accessories.urdf.xacro"/>
   <xacro:include filename="$(find clearpath_sensors_description)/urdf/intel_realsense.urdf.xacro"/>
   <material name="black">
@@ -14,5 +14,5 @@
       <material name="black"/>
       <geometry>
-        <mesh filename="package://lab_manipulator/meshes/mounting_structure.STL"/>
+        <mesh filename="package://claus/meshes/mounting_structure.STL"/>
       </geometry>
     </visual>
@@ -20,5 +20,5 @@
       <origin xyz="0 0 0" rpy="0 0 0"/>
       <geometry>
-        <mesh filename="package://lab_manipulator/meshes/mounting_structure.STL"/>
+        <mesh filename="package://claus/meshes/mounting_structure.STL"/>
       </geometry>
     </collision>
@@ -74,5 +74,5 @@
       <origin xyz="0.02 0 0" rpy="${pi/2} 1.0471975512 ${pi/2}" />
       <geometry>
-        <mesh filename="package://lab_manipulator/meshes/d435.dae" />
+        <mesh filename="package://claus/meshes/d435.dae" />
       </geometry>
       <material name="white" />
